Commit message: urdf_sans_camera

File: install/V1_Robot_Mobil_description/share/V1_Robot_Mobil_description/urdf/V1_Robot_Mobil.xacro (robot description, xacro)
@@ -912,5 +912,5 @@
   </collision>
 </link> -->
-<link name="Camera_stereo_v3_1">
+<!-- <link name="Camera_stereo_v3_1">
   <inertial>
     <origin xyz="-0.03749953126062 0.007467405126430793 -0.007104288060535674" rpy="0 0 0"/>
@@ -931,5 +931,5 @@
     </geometry>
   </collision>
-</link>
+</link> -->
 <link name="illustation_entretoise_12mm_v2__8__1">
   <inertial>
@@ -1292,4 +1292,5 @@
   </collision>
 </link>
+<!--
 <link name="support_camera_stereo">
   <inertial>
@@ -1311,5 +1312,5 @@
     </geometry>
   </collision>
-</link>
+</link> -->
 <link name="world"/>
 <joint name="base_joint" type="fixed">
@@ -1429,14 +1430,15 @@
   <child link="illustation_entretoise_12mm_v2__2__1"/>
 </joint> -->
-<joint name="Rigide 31" type="fixed">
+<!-- <joint name="Rigide 31" type="fixed">
   <origin xyz="-0.024834 0.139481 0.069149" rpy="0 0 0"/>
   <parent link="base_link"/>
   <child link="Camera_stereo_v3_1"/>
-</joint>
+</joint> -->
+<!--
 <joint name="Support_Camera" type="fixed">
   <origin xyz="-0.0 -0.000 0.0" rpy="0 0 0"/>
   <parent link="base_link"/>
   <child link="support_camera_stereo"/>
-</joint>
+</joint> -->
 <!-- <joint name="Rigide 32" type="fixed">
   <origin xyz="0.0 0.0 0.012" rpy="0 0 0"/>

Commit message: add lidar plugin

File: install/V1_Robot_Mobil_description/share/V1_Robot_Mobil_description/urdf/V1_Robot_Mobil.xacro (robot description, xacro)
@@ -3,5 +3,17 @@
 <xacro:include filename="$(find V1_Robot_Mobil_description)/urdf/materials.xacro" />
 <xacro:include filename="$(find V1_Robot_Mobil_description)/urdf/V1_Robot_Mobil.trans" />
-<!-- <xacro:include filename="$(find V1_Robot_Mobil_description)/urdf/V1_Robot_Mobil_gazebo" />  -->
+<xacro:include filename="$(find V1_Robot_Mobil_description)/urdf/V1_Robot_Mobil_gazebo.xacro" />
+<xacro:property name="laser_LIDAR_part2_v2_1_offsety" value="0"/>
+<xacro:property name="LIDAR_part2_v2_1_LIDAR_part1_v4_1_offsety" value="0.04199"/>
+<xacro:property name="LIDAR_part1_v4_1_illustation_entretoise_12mm_v2__8__1_offsety" value="0"/>
+<xacro:property name="illustation_entretoise_12mm_v2__8__1_lidarPlate_v6_1_offsety" value="0.0104"/>
+<xacro:property name="lidarPlate_v6_1_illustation_entretoise_70mm_v1_1_offsety" value="0"/>
+<xacro:property name="illustation_entretoise_70mm_v1_1_base_link_offsety" value="-0.075019"/>
+<xacro:property name="Roue_droite_1_gente_gauche_1_offsety" value="0"/>
+<xacro:property name="gente_gauche_1_moteur_jaune_1_offsety" value="0.0206"/>
+<xacro:property name="moteur_jaune_1_support_roue_2_offsety" value="0"/>
+<xacro:property name="support_roue_2_base_link_offsety" value="-0.000519"/>
+<xacro:property name="laser_base_link_offsety" value="${laser_LIDAR_part2_v2_1_offsety + LIDAR_part2_v2_1_LIDAR_part1_v4_1_offsety + LIDAR_part1_v4_1_illustation_entretoise_12mm_v2__8__1_offsety + illustation_entretoise_12mm_v2__8__1_lidarPlate_v6_1_offsety + lidarPlate_v6_1_illustation_entretoise_70mm_v1_1_offsety + illustation_entretoise_70mm_v1_1_base_link_offsety}"/>
+<xacro:property name="Roue_droite_1_base_link_offsety" value="${Roue_droite_1_gente_gauche_1_offsety + gente_gauche_1_moteur_jaune_1_offsety + moteur_jaune_1_support_roue_2_offsety + support_roue_2_base_link_offsety}"/>
 <link name="base_link">
   <inertial>
@@ -184,312 +196,4 @@
   </collision>
 </link>
-<!--
-<link name="SG90_V1_v1_1">
-  <inertial>
-    <origin xyz="0.03487746847113202 0.014544287043435106 -0.06161565969845402" rpy="0 0 0"/>
-    <mass value="0.047113050905792125"/>
-    <inertia ixx="4e-06" iyy="3e-06" izz="3e-06" ixy="-0.0" iyz="-0.0" ixz="0.0"/>
-  </inertial>
-  <visual>
-    <origin xyz="0.046211 -0.090448 -0.135298" rpy="0 0 0"/>
-    <geometry>
-      <mesh filename="file://$(find V1_Robot_Mobil_description)/meshes/SG90_V1_v1_1.stl" scale="0.001 0.001 0.001"/>
-    </geometry>
-    <material name="silver"/>
-  </visual>
-  <collision>
-    <origin xyz="0.046211 -0.090448 -0.135298" rpy="0 0 0"/>
-    <geometry>
-      <mesh filename="file://$(find V1_Robot_Mobil_description)/meshes/SG90_V1_v1_1.stl" scale="0.001 0.001 0.001"/>
-    </geometry>
-  </collision>
-</link> -->
-<!-- <link name="illustation_entretoise_12mm_v2_1">
-  <inertial>
-    <origin xyz="4.6847145871234397e-07 2.323489760036601e-07 0.006000057369971307" rpy="0 0 0"/>
-    <mass value="0.0006394129256555783"/>
-    <inertia ixx="0.0" iyy="0.0" izz="0.0" ixy="0.0" iyz="-0.0" ixz="0.0"/>
-  </inertial>
-  <visual>
-    <origin xyz="0.024834 -0.119481 -0.069149" rpy="0 0 0"/>
-    <geometry>
-      <mesh filename="file://$(find V1_Robot_Mobil_description)/meshes/illustation_entretoise_12mm_v2_1.stl" scale="0.001 0.001 0.001"/>
-    </geometry>
-    <material name="silver"/>
-  </visual>
-  <collision>
-    <origin xyz="0.024834 -0.119481 -0.069149" rpy="0 0 0"/>
-    <geometry>
-      <mesh filename="file://$(find V1_Robot_Mobil_description)/meshes/illustation_entretoise_12mm_v2_1.stl" scale="0.001 0.001 0.001"/>
-    </geometry>
-  </collision>
-</link> -->
-<!-- <link name="illustation_entretoise_12mm_v2__1__1">
-  <inertial>
-    <origin xyz="4.6847145873359433e-07 2.3234897604529348e-07 0.00600005736997139" rpy="0 0 0"/>
-    <mass value="0.0006394129256555783"/>
-    <inertia ixx="0.0" iyy="0.0" izz="0.0" ixy="-0.0" iyz="0.0" ixz="-0.0"/>
-  </inertial>
-  <visual>
-    <origin xyz="-0.002166 -0.119481 -0.069149" rpy="0 0 0"/>
-    <geometry>
-      <mesh filename="file://$(find V1_Robot_Mobil_description)/meshes/illustation_entretoise_12mm_v2__1__1.stl" scale="0.001 0.001 0.001"/>
-    </geometry>
-    <material name="silver"/>
-  </visual>
-  <collision>
-    <origin xyz="-0.002166 -0.119481 -0.069149" rpy="0 0 0"/>
-    <geometry>
-      <mesh filename="file://$(find V1_Robot_Mobil_description)/meshes/illustation_entretoise_12mm_v2__1__1.stl" scale="0.001 0.001 0.001"/>
-    </geometry>
-  </collision>
-</link> -->
-<!-- <link name="illustation_entretoise_12mm_v2__2__1">
-  <inertial>
-    <origin xyz="4.684714587067061e-07 2.3234897592039339e-07 0.00600005736997139" rpy="0 0 0"/>
-    <mass value="0.0006394129256555783"/>
-    <inertia ixx="0.0" iyy="0.0" izz="0.0" ixy="-0.0" iyz="-0.0" ixz="-0.0"/>
-  </inertial>
-  <visual>
-    <origin xyz="-0.002166 -0.139481 -0.069149" rpy="0 0 0"/>
-    <geometry>
-      <mesh filename="file://$(find V1_Robot_Mobil_description)/meshes/illustation_entretoise_12mm_v2__2__1.stl" scale="0.001 0.001 0.001"/>
-    </geometry>
-    <material name="silver"/>
-  </visual>
-  <collision>
-    <origin xyz="-0.002166 -0.139481 -0.069149" rpy="0 0 0"/>
-    <geometry>
-      <mesh filename="file://$(find V1_Robot_Mobil_description)/meshes/illustation_entretoise_12mm_v2__2__1.stl" scale="0.001 0.001 0.001"/>
-    </geometry>
-  </collision>
-</link> -->
-<!-- <link name="illustation_entretoise_12mm_v2__3__1">
-  <inertial>
-    <origin xyz="4.684714586776495e-07 2.3234897594814896e-07 0.006000057369971334" rpy="0 0 0"/>
-    <mass value="0.0006394129256555783"/>
-    <inertia ixx="0.0" iyy="0.0" izz="0.0" ixy="0.0" iyz="-0.0" ixz="0.0"/>
-  </inertial>
-  <visual>
-    <origin xyz="0.024834 -0.139481 -0.069149" rpy="0 0 0"/>
-    <geometry>
-      <mesh filename="file://$(find V1_Robot_Mobil_description)/meshes/illustation_entretoise_12mm_v2__3__1.stl" scale="0.001 0.001 0.001"/>
-    </geometry>
-    <material name="silver"/>
-  </visual>
-  <collision>
-    <origin xyz="0.024834 -0.139481 -0.069149" rpy="0 0 0"/>
-    <geometry>
-      <mesh filename="file://$(find V1_Robot_Mobil_description)/meshes/illustation_entretoise_12mm_v2__3__1.stl" scale="0.001 0.001 0.001"/>
-    </geometry>
-  </collision>
-</link> -->
-<!--
-<link name="Socle_Niv1_v6_1">
-  <inertial>
-    <origin xyz="-0.013629751684390345 -0.009999767720685976 0.0010000573699713577" rpy="0 0 0"/>
-    <mass value="0.017490216835436147"/>
-    <inertia ixx="1e-06" iyy="6e-06" izz="7e-06" ixy="0.0" iyz="0.0" ixz="0.0"/>
-  </inertial>
-  <visual>
-    <origin xyz="-0.002166 -0.139481 -0.081149" rpy="0 0 0"/>
-    <geometry>
-      <mesh filename="file://$(find V1_Robot_Mobil_description)/meshes/Socle_Niv1_v6_1.stl" scale="0.001 0.001 0.001"/>
-    </geometry>
-    <material name="silver"/>
-  </visual>
-  <collision>
-    <origin xyz="-0.002166 -0.139481 -0.081149" rpy="0 0 0"/>
-    <geometry>
-      <mesh filename="file://$(find V1_Robot_Mobil_description)/meshes/Socle_Niv1_v6_1.stl" scale="0.001 0.001 0.001"/>
-    </geometry>
-  </collision>
-</link> -->
-<!-- <link name="illustation_entretoise_3_v2_1">
-  <inertial>
-    <origin xyz="4.687395950171702e-07 2.3234897586488223e-07 0.004000057369971374" rpy="0 0 0"/>
-    <mass value="0.00017036001397236956"/>
-    <inertia ixx="0.0" iyy="0.0" izz="0.0" ixy="-0.0" iyz="0.0" ixz="0.0"/>
-  </inertial>
-  <visual>
-    <origin xyz="0.025134 -0.129481 -0.083149" rpy="0 0 0"/>
-    <geometry>
-      <mesh filename="file://$(find V1_Robot_Mobil_description)/meshes/illustation_entretoise_3_v2_1.stl" scale="0.001 0.001 0.001"/>
-    </geometry>
-    <material name="silver"/>
-  </visual>
-  <collision>
-    <origin xyz="0.025134 -0.129481 -0.083149" rpy="0 0 0"/>
-    <geometry>
-      <mesh filename="file://$(find V1_Robot_Mobil_description)/meshes/illustation_entretoise_3_v2_1.stl" scale="0.001 0.001 0.001"/>
-    </geometry>
-  </collision>
-</link> -->
-<!--
-<link name="illustation_entretoise_3_v2__1__1">
-  <inertial>
-    <origin xyz="4.6908232182460777e-07 2.323489758926378e-07 0.004000057369971374" rpy="0 0 0"/>
-    <mass value="0.00017036001397236956"/>
-    <inertia ixx="0.0" iyy="0.0" izz="0.0" ixy="-0.0" iyz="0.0" ixz="-0.0"/>
-  </inertial>
-  <visual>
-    <origin xyz="-0.003466 -0.129481 -0.083149" rpy="0 0 0"/>
-    <geometry>
-      <mesh filename="file://$(find V1_Robot_Mobil_description)/meshes/illustation_entretoise_3_v2__1__1.stl" scale="0.001 0.001 0.001"/>
-    </geometry>
-    <material name="silver"/>
-  </visual>
-  <collision>
-    <origin xyz="-0.003466 -0.129481 -0.083149" rpy="0 0 0"/>
-    <geometry>
-      <mesh filename="file://$(find V1_Robot_Mobil_description)/meshes/illustation_entretoise_3_v2__1__1.stl" scale="0.001 0.001 0.001"/>
-    </geometry>
-  </collision>
-</link> -->
-<!--
-<link name="SG90_V1_v1__1__1">
-  <inertial>
-    <origin xyz="0.013811523433811939 2.323489758926378e-07 -0.002033225561603305" rpy="0 0 0"/>
-    <mass value="0.047113050905792125"/>
-    <inertia ixx="3e-06" iyy="4e-06" izz="3e-06" ixy="-0.0" iyz="0.0" ixz="0.0"/>
-  </inertial>
-  <visual>
-    <origin xyz="0.025134 -0.129481 -0.091149" rpy="0 0 0"/>
-    <geometry>
-      <mesh filename="file://$(find V1_Robot_Mobil_description)/meshes/SG90_V1_v1__1__1.stl" scale="0.001 0.001 0.001"/>
-    </geometry>
-    <material name="silver"/>
-  </visual>
-  <collision>
-    <origin xyz="0.025134 -0.129481 -0.091149" rpy="0 0 0"/>
-    <geometry>
-      <mesh filename="file://$(find V1_Robot_Mobil_description)/meshes/SG90_V1_v1__1__1.stl" scale="0.001 0.001 0.001"/>
-    </geometry>
-  </collision>
-</link> -->
-<!--
-<link name="SG90_slot_1_1">
-  <inertial>
-    <origin xyz="4.6873400406238774e-07 2.3285903644199024e-07 0.00214911116079651" rpy="0 0 0"/>
-    <mass value="0.0014672674655415944"/>
-    <inertia ixx="1e-08" iyy="6e-08" izz="6e-08" ixy="-0.0" iyz="0.0" ixz="-0.0"/>
-  </inertial>
-  <visual>
-    <origin xyz="0.015934 -0.129481 -0.101949" rpy="0 0 0"/>
-    <geometry>
-      <mesh filename="file://$(find V1_Robot_Mobil_description)/meshes/SG90_slot_1_1.stl" scale="0.001 0.001 0.001"/>
-    </geometry>
-    <material name="silver"/>
-  </visual>
-  <collision>
-    <origin xyz="0.015934 -0.129481 -0.101949" rpy="0 0 0"/>
-    <geometry>
-      <mesh filename="file://$(find V1_Robot_Mobil_description)/meshes/SG90_slot_1_1.stl" scale="0.001 0.001 0.001"/>
-    </geometry>
-  </collision>
-</link> -->
-<!--
-<link name="base_camera_niv1_v1_1">
-  <inertial>
-    <origin xyz="4.675759468497631e-07 2.3209993837980392e-07 -0.0009999426300286302" rpy="0 0 0"/>
-    <mass value="0.04794063452340887"/>
-    <inertia ixx="3e-06" iyy="5.8e-05" izz="6.1e-05" ixy="-0.0" iyz="0.0" ixz="0.0"/>
-  </inertial>
-  <visual>
-    <origin xyz="0.015934 -0.129481 -0.103949" rpy="0 0 0"/>
-    <geometry>
-      <mesh filename="file://$(find V1_Robot_Mobil_description)/meshes/base_camera_niv1_v1_1.stl" scale="0.001 0.001 0.001"/>
-    </geometry>
-    <material name="silver"/>
-  </visual>
-  <collision>
-    <origin xyz="0.015934 -0.129481 -0.103949" rpy="0 0 0"/>
-    <geometry>
-      <mesh filename="file://$(find V1_Robot_Mobil_description)/meshes/base_camera_niv1_v1_1.stl" scale="0.001 0.001 0.001"/>
-    </geometry>
-  </collision>
-</link> -->
-<!--
-<link name="base_camera_niv2_1_v6_1">
-  <inertial>
-    <origin xyz="4.687393527769146e-07 -0.006999173760916216 0.0172982109600035" rpy="0 0 0"/>
-    <mass value="0.014155958827538562"/>
-    <inertia ixx="2e-06" iyy="1e-06" izz="1e-06" ixy="-0.0" iyz="0.0" ixz="0.0"/>
-  </inertial>
-  <visual>
-    <origin xyz="0.071434 -0.136481 -0.103949" rpy="0 0 0"/>
-    <geometry>
-      <mesh filename="file://$(find V1_Robot_Mobil_description)/meshes/base_camera_niv2_1_v6_1.stl" scale="0.001 0.001 0.001"/>
-    </geometry>
-    <material name="silver"/>
-  </visual>
-  <collision>
-    <origin xyz="0.071434 -0.136481 -0.103949" rpy="0 0 0"/>
-    <geometry>
-      <mesh filename="file://$(find V1_Robot_Mobil_description)/meshes/base_camera_niv2_1_v6_1.stl" scale="0.001 0.001 0.001"/>
-    </geometry>
-  </collision>
-</link> -->
-<!--
-<link name="base_camera_niv2_2_v5_1">
-  <inertial>
-    <origin xyz="4.6873935293650915e-07 0.006999441294755826 0.016570769687492798" rpy="0 0 0"/>
-    <mass value="0.010627696385805586"/>
-    <inertia ixx="2e-06" iyy="1e-06" izz="1e-06" ixy="-0.0" iyz="-0.0" ixz="0.0"/>
-  </inertial>
-  <visual>
-    <origin xyz="-0.039566 -0.122481 -0.103949" rpy="0 0 0"/>
-    <geometry>
-      <mesh filename="file://$(find V1_Robot_Mobil_description)/meshes/base_camera_niv2_2_v5_1.stl" scale="0.001 0.001 0.001"/>
-    </geometry>
-    <material name="silver"/>
-  </visual>
-  <collision>
-    <origin xyz="-0.039566 -0.122481 -0.103949" rpy="0 0 0"/>
-    <geometry>
-      <mesh filename="file://$(find V1_Robot_Mobil_description)/meshes/base_camera_niv2_2_v5_1.stl" scale="0.001 0.001 0.001"/>
-    </geometry>
-  </collision>
-</link> -->
-<!-- <link name="SG90_V1_v1__2__1">
-  <inertial>
-    <origin xyz="-0.004532814192221665 0.013811287043434956 3.8157455434228993e-07" rpy="0 0 0"/>
-    <mass value="0.047113050905792125"/>
-    <inertia ixx="3e-06" iyy="3e-06" izz="4e-06" ixy="0.0" iyz="-0.0" ixz="0.0"/>
-  </inertial>
-  <visual>
-    <origin xyz="-0.038566 -0.115281 -0.123438" rpy="0 0 0"/>
-    <geometry>
-      <mesh filename="file://$(find V1_Robot_Mobil_description)/meshes/SG90_V1_v1__2__1.stl" scale="0.001 0.001 0.001"/>
-    </geometry>
-    <material name="silver"/>
-  </visual>
-  <collision>
-    <origin xyz="-0.038566 -0.115281 -0.123438" rpy="0 0 0"/>
-    <geometry>
-      <mesh filename="file://$(find V1_Robot_Mobil_description)/meshes/SG90_V1_v1__2__1.stl" scale="0.001 0.001 0.001"/>
-    </geometry>
-  </collision>
-</link> -->
-<!-- <link name="slot_type_2_v4_1">
-  <inertial>
-    <origin xyz="0.002002547906652566 -9.760176477566218e-06 0.002672180343408617" rpy="0 0 0"/>
-    <mass value="0.0011011067412301362"/>
-    <inertia ixx="3e-08" iyy="2e-08" izz="1e-08" ixy="0.0" iyz="-0.0" ixz="-0.0"/>
-  </inertial>
-  <visual>
-    <origin xyz="-0.046866 -0.124481 -0.123438" rpy="0 0 0"/>
-    <geometry>
-      <mesh filename="file://$(find V1_Robot_Mobil_description)/meshes/slot_type_2_v4_1.stl" scale="0.001 0.001 0.001"/>
-    </geometry>
-    <material name="silver"/>
-  </visual>
-  <collision>
-    <origin xyz="-0.046866 -0.124481 -0.123438" rpy="0 0 0"/>
-    <geometry>
-      <mesh filename="file://$(find V1_Robot_Mobil_description)/meshes/slot_type_2_v4_1.stl" scale="0.001 0.001 0.001"/>
-    </geometry>
-  </collision>
-</link> -->
 <link name="illustation_entretoise_70mm_v1_1">
   <inertial>
@@ -852,84 +556,4 @@
   </collision>
 </link>
-<!-- <link name="base_camera_niv3_1_v2_1">
-  <inertial>
-    <origin xyz="0.12148846873935296 0.12461633307319951 0.060378864280039635" rpy="0 0 0"/>
-    <mass value="0.006793511398361307"/>
-    <inertia ixx="1e-06" iyy="1e-06" izz="0.0" ixy="0.0" iyz="-0.0" ixz="0.0"/>
-  </inertial>
-  <visual>
-    <origin xyz="0.073572 -0.0 -0.076572" rpy="0 0 0"/>
-    <geometry>
-      <mesh filename="file://$(find V1_Robot_Mobil_description)/meshes/base_camera_niv3_1_v2_1.stl" scale="0.001 0.001 0.001"/>
-    </geometry>
-    <material name="silver"/>
-  </visual>
-  <collision>
-    <origin xyz="0.073572 -0.0 -0.076572" rpy="0 0 0"/>
-    <geometry>
-      <mesh filename="file://$(find V1_Robot_Mobil_description)/meshes/base_camera_niv3_1_v2_1.stl" scale="0.001 0.001 0.001"/>
-    </geometry>
-  </collision>
-</link> -->
-<!-- <link name="base_camera_niv3_v4_1">
-  <inertial>
-    <origin xyz="0.09864446873935112 0.050959232348975855 -0.10744265137903988" rpy="0 0 0"/>
-    <mass value="0.10377906280662101"/>
-    <inertia ixx="8e-06" iyy="0.000115" izz="0.000108" ixy="0.0" iyz="0.0" ixz="0.0"/>
-  </inertial>
-  <visual>
-    <origin xyz="0.107478 -0.073522 -0.259328" rpy="0 0 0"/>
-    <geometry>
-      <mesh filename="file://$(find V1_Robot_Mobil_description)/meshes/base_camera_niv3_v4_1.stl" scale="0.001 0.001 0.001"/>
-    </geometry>
-    <material name="silver"/>
-  </visual>
-  <collision>
-    <origin xyz="0.107478 -0.073522 -0.259328" rpy="0 0 0"/>
-    <geometry>
-      <mesh filename="file://$(find V1_Robot_Mobil_description)/meshes/base_camera_niv3_v4_1.stl" scale="0.001 0.001 0.001"/>
-    </geometry>
-  </collision>
-</link> -->
-<!-- <link name="base_camera_niv3_1_v2__1__1">
-  <inertial>
-    <origin xyz="0.008478468739352998 0.1552793330731995 -0.14284313571996035" rpy="0 0 0"/>
-    <mass value="0.006793511398361307"/>
-    <inertia ixx="1e-06" iyy="1e-06" izz="0.0" ixy="0.0" iyz="-0.0" ixz="-0.0"/>
-  </inertial>
-  <visual>
-    <origin xyz="0.073562 0.030663 -0.279794" rpy="0 0 0"/>
-    <geometry>
-      <mesh filename="file://$(find V1_Robot_Mobil_description)/meshes/base_camera_niv3_1_v2__1__1.stl" scale="0.001 0.001 0.001"/>
-    </geometry>
-    <material name="silver"/>
-  </visual>
-  <collision>
-    <origin xyz="0.073562 0.030663 -0.279794" rpy="0 0 0"/>
-    <geometry>
-      <mesh filename="file://$(find V1_Robot_Mobil_description)/meshes/base_camera_niv3_1_v2__1__1.stl" scale="0.001 0.001 0.001"/>
-    </geometry>
-  </collision>
-</link> -->
-<!-- <link name="Camera_stereo_v3_1">
-  <inertial>
-    <origin xyz="-0.03749953126062 0.007467405126430793 -0.007104288060535674" rpy="0 0 0"/>
-    <mass value="0.28987792909524945"/>
-    <inertia ixx="2.4e-05" iyy="0.000209" izz="0.000196" ixy="0.0" iyz="0.0" ixz="-0.0"/>
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
File: install/V1_Robot_Mobil_description/share/V1_Robot_Mobil_description/urdf/V1_Robot_Mobil_gazebo.xacro (robot description, xacro)
@@ -2,26 +2,47 @@
 <robot xmlns:xacro="http://www.ros.org/wiki/xacro" >
 <xacro:property name="body_color" value="Gazebo/Silver" />
-<!--
-<gazebo>
-  <plugin name="control" filename="libgazebo_ros_control.so"/>
-</gazebo> -->
 <gazebo>
         <plugin
             filename="gz-sim-diff-drive-system"
             name="gz::sim::systems::DiffDrive">
-            <left_joint>Revolution 24</left_joint>
-            <right_joint>Revolution 25</right_joint>
+            <left_joint>revolution 24</left_joint>
+            <right_joint>revolution 25</right_joint>
             <wheel_separation>0.45</wheel_separation>
             <wheel_radius>0.1</wheel_radius>
             <frame_id>odom</frame_id>
-            <child_frame_id>world</child_frame_id>
+            <child_frame_id>base_footprint</child_frame_id>
         </plugin>
-    </gazebo>
-    <gazebo>
+</gazebo>
+<gazebo reference="LIDAR_part2_v2_1">
+  <sensor type="gpu_lidar" name="gpu_lidar">
+    <update_rate>10</update_rate>
+    <ray>
+      <scan>
+        <horizontal>
+          <samples>360</samples>
+          <resolution>1</resolution>
+          <min_angle>-3.14</min_angle>
+          <max_angle>3.14</max_angle>
+        </horizontal>
+      </scan>
+      <range>
+        <min>0.1</min>
+        <max>10.0</max>
+        <resolution>0.01</resolution>
+      </range>
+    </ray>
+    <visualize> true </visualize>
+    <plugin name="gz::sim::systems::Sensors" filename="gz-sim-sensors-system">
+      <topicName>/scan</topicName>
+      <frameName>base_footprint</frameName>
+    </plugin>
+  </sensor>
+</gazebo>
+<gazebo>
         <plugin
             filename="gz-sim-joint-state-publisher-system"
             name="gz::sim::systems::JointStatePublisher">
-            <joint_name>Revolution 24</joint_name>
-            <joint_name>Revolution 25</joint_name>
+            <joint_name>revolution 24</joint_name>
+            <joint_name>revolution 25</joint_name>
         </plugin>
 </gazebo>
